Commit message: 手动修改文件，更新任务进度

File: workspaces/ws_tutorials/src/ur3_joint_state_publisher_py/urdf/ur3_simplified.urdf.xacro (robot description, xacro)
@@ -3,9 +3,11 @@
   <xacro:arg name="link_2_length" default="0.34"/>
   <xacro:arg name="tool0_offset_z" default="0.12"/>
-  <xacro:arg name="joint_limit_scale" default="1.0"/>
+  <xacro:arg name="upper_joint_limit_scale" default="1.0"/>
+  <xacro:arg name="lower_joint_limit_scale" default="1.0"/>
   <xacro:include filename="$(find ur3_joint_state_publisher_py)/urdf/ur3_simplified_macro.xacro"/>
   <xacro:ur3_simplified_chain
     link_2_length="$(arg link_2_length)"
     tool0_offset_z="$(arg tool0_offset_z)"
-    joint_limit_scale="$(arg joint_limit_scale)"/>
+    upper_joint_limit_scale="$(arg upper_joint_limit_scale)"
+    lower_joint_limit_scale="$(arg lower_joint_limit_scale)"/>
 </robot>

File: workspaces/ws_tutorials/src/ur3_joint_state_publisher_py/urdf/ur3_simplified_macro.xacro (robot description, xacro)
@@ -4,7 +4,9 @@
       link_2_length:=0.34
       tool0_offset_z:=0.12
-      joint_limit_scale:=1.0">
+      upper_joint_limit_scale:=1.0
+      lower_joint_limit_scale:=1.0">
     <!-- TODO(human): Decide whether to expose per-joint lower/upper limits instead of one global scale. -->
-    <xacro:property name="joint_limit_rad" value="${3.14 * joint_limit_scale}"/>
+    <xacro:property name="upper_joint_limit_rad" value="${3.14 * upper_joint_limit_scale}"/>
+    <xacro:property name="lower_joint_limit_rad" value="${3.14 * lower_joint_limit_scale}"/>
     <material name="steel_gray">
       <color rgba="0.60 0.62 0.66 1.0"/>
@@ -93,5 +95,5 @@
       <origin xyz="0 0 0.08" rpy="0 0 0"/>
       <axis xyz="0 0 1"/>
-      <limit lower="${-joint_limit_rad}" upper="${joint_limit_rad}" effort="50.0" velocity="2.0"/>
+      <limit lower="${-lower_joint_limit_rad}" upper="${upper_joint_limit_rad}" effort="50.0" velocity="2.0"/>
     </joint>
     <joint name="shoulder_lift_joint" type="revolute">
@@ -100,5 +102,5 @@
       <origin xyz="0 0 0.20" rpy="0 0 0"/>
       <axis xyz="0 1 0"/>
-      <limit lower="${-joint_limit_rad}" upper="${joint_limit_rad}" effort="50.0" velocity="2.0"/>
+      <limit lower="${-lower_joint_limit_rad}" upper="${upper_joint_limit_rad}" effort="50.0" velocity="2.0"/>
     </joint>
     <joint name="elbow_joint" type="revolute">
@@ -107,5 +109,5 @@
       <origin xyz="0 0 ${link_2_length}" rpy="0 0 0"/>
       <axis xyz="0 1 0"/>
-      <limit lower="${-joint_limit_rad}" upper="${joint_limit_rad}" effort="40.0" velocity="2.2"/>
+      <limit lower="${-lower_joint_limit_rad}" upper="${upper_joint_limit_rad}" effort="40.0" velocity="2.2"/>
     </joint>
     <joint name="wrist_1_joint" type="revolute">
@@ -114,5 +116,5 @@
       <origin xyz="0 0 0.30" rpy="0 0 0"/>
       <axis xyz="0 1 0"/>
-      <limit lower="${-joint_limit_rad}" upper="${joint_limit_rad}" effort="25.0" velocity="2.5"/>
+      <limit lower="${-lower_joint_limit_rad}" upper="${upper_joint_limit_rad}" effort="25.0" velocity="2.5"/>
     </joint>
     <joint name="wrist_2_joint" type="revolute">
@@ -121,5 +123,5 @@
       <origin xyz="0 0 0.20" rpy="0 0 0"/>
       <axis xyz="0 0 1"/>
-      <limit lower="${-joint_limit_rad}" upper="${joint_limit_rad}" effort="20.0" velocity="2.8"/>
+      <limit lower="${-lower_joint_limit_rad}" upper="${upper_joint_limit_rad}" effort="20.0" velocity="2.8"/>
     </joint>
     <joint name="wrist_3_joint" type="revolute">
@@ -128,5 +130,5 @@
       <origin xyz="0 0 0.16" rpy="0 0 0"/>
       <axis xyz="0 1 0"/>
-      <limit lower="${-joint_limit_rad}" upper="${joint_limit_rad}" effort="15.0" velocity="3.0"/>
+      <limit lower="${-lower_joint_limit_rad}" upper="${upper_joint_limit_rad}" effort="15.0" velocity="3.0"/>
     </joint>
     <joint name="tool0_fixed_joint" type="fixed">
